File: pcb/keyboard_shortcut_board.kicad_sch (KiCad schematic)
At the start: 30 parts, among them SW1 SW_Push, SW10 RotaryEncoder, SW2 SW_Push, SW3 SW_Push, SW4 SW_Push, SW5 SW_Push, SW6 SW_Push, SW7 SW_Push, SW8 SW_Push, SW9 SW_Push, U1 MOUDLE-SEEEDUINO-XIAO, U2 ER_OLEDM0.91_1x-I2C

Commit message: fix schematic power rails
Connections:
- net GND: now reaches D1.3 (VSS), D2.3 (VSS), D3.3 (VSS), D4.3 (VSS), D5.3 (VSS), D6.3 (VSS), D7.3 (VSS), D8.3 (VSS), D9.3 (VSS), SW10.C, U1.13 (GND), U2.1 (GND)
- net +5V: now reaches D1.1 (VDD), D2.1 (VDD), D3.1 (VDD), D4.1 (VDD), D5.1 (VDD), D6.1 (VDD), D7.1 (VDD), D8.1 (VDD), D9.1 (VDD)
- net +5V: now also U1.14 (5V), U2.2 (VCC); no longer U1.12 (3V3)
- no-connect marks 0 -> 2
